File: nixie2.sch (KiCad schematic (older format))
At the start: 46 parts, among them J1 AVR-ISP-6, J14 Conn_01x10_Female, SW1 Conn_01x02_Male, SW2 Conn_01x02_Male, SW3 Conn_01x02_Male, SW4 Conn_01x02_Male, SW5 Conn_01x02_Male, SW6 Conn_01x02_Male, U1 ATmega8-16PU, U10 74141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

Commit message: Add tube adapter board, and tweak main board
Parts:
- R2, R3, R4, R5, R6, R7: footprint Resistor_THT:R_Axial_DIN0207_L6.3mm_D2.5mm_P2.54mm_Vertical -> Resistor_THT:R_Axial_DIN0207_L6.3mm_D2.5mm_P7.62mm_Horizontal
Changed lines of the file:
@@
 F 0 "R5" V 3595 12450 50  0000 C CNN
 F 1 "10k" V 3686 12450 50  0000 C CNN
-F 2 "Resistor_THT:R_Axial_DIN0207_L6.3mm_D2.5mm_P2.54mm_Vertical" V 3840 12440 50  0001 C CNN
+F 2 "Resistor_THT:R_Axial_DIN0207_L6.3mm_D2.5mm_P7.62mm_Horizontal" V 3840 12440 50  0001 C CNN
 F 3 "~" H 3800 12450 50  0001 C CNN
 	1    3800 12450
@@
 F 0 "R6" V 3595 12750 50  0000 C CNN
 F 1 "10k" V 3686 12750 50  0000 C CNN
-F 2 "Resistor_THT:R_Axial_DIN0207_L6.3mm_D2.5mm_P2.54mm_Vertical" V 3840 12740 50  0001 C CNN
+F 2 "Resistor_THT:R_Axial_DIN0207_L6.3mm_D2.5mm_P7.62mm_Horizontal" V 3840 12740 50  0001 C CNN
 F 3 "~" H 3800 12750 50  0001 C CNN
 	1    3800 12750
@@
 F 0 "R4" V 3595 12150 50  0000 C CNN
 F 1 "10k" V 3686 12150 50  0000 C CNN
-F 2 "Resistor_THT:R_Axial_DIN0207_L6.3mm_D2.5mm_P2.54mm_Vertical" V 3840 12140 50  0001 C CNN
+F 2 "Resistor_THT:R_Axial_DIN0207_L6.3mm_D2.5mm_P7.62mm_Horizontal" V 3840 12140 50  0001 C CNN
 F 3 "~" H 3800 12150 50  0001 C CNN
 	1    3800 12150
@@
 F 0 "R3" V 3595 11900 50  0000 C CNN
 F 1 "10k" V 3686 11900 50  0000 C CNN
-F 2 "Resistor_THT:R_Axial_DIN0207_L6.3mm_D2.5mm_P2.54mm_Vertical" V 3840 11890 50  0001 C CNN
+F 2 "Resistor_THT:R_Axial_DIN0207_L6.3mm_D2.5mm_P7.62mm_Horizontal" V 3840 11890 50  0001 C CNN
 F 3 "~" H 3800 11900 50  0001 C CNN
 	1    3800 11900
@@
 F 0 "R7" V 3595 13000 50  0000 C CNN
 F 1 "10k" V 3686 13000 50  0000 C CNN
-F 2 "Resistor_THT:R_Axial_DIN0207_L6.3mm_D2.5mm_P2.54mm_Vertical" V 3840 12990 50  0001 C CNN
+F 2 "Resistor_THT:R_Axial_DIN0207_L6.3mm_D2.5mm_P7.62mm_Horizontal" V 3840 12990 50  0001 C CNN
 F 3 "~" H 3800 13000 50  0001 C CNN
 	1    3800 13000
@@
 F 0 "R2" V 3595 11650 50  0000 C CNN
 F 1 "10k" V 3686 11650 50  0000 C CNN
-F 2 "Resistor_THT:R_Axial_DIN0207_L6.3mm_D2.5mm_P2.54mm_Vertical" V 3840 11640 50  0001 C CNN
+F 2 "Resistor_THT:R_Axial_DIN0207_L6.3mm_D2.5mm_P7.62mm_Horizontal" V 3840 11640 50  0001 C CNN
 F 3 "~" H 3800 11650 50  0001 C CNN
 	1    3800 11650
