File: nixie2.kicad_pcb (KiCad board)
At the start: 2 copper layers, 68.5 x 181 mm, 51 parts, among them J1 AVR-ISP-6, J14 Conn_01x10_Female, SW1 Conn_01x02_Male, SW2 Conn_01x02_Male, SW3 Conn_01x02_Male, SW4 Conn_01x02_Male, SW5 Conn_01x02_Male, SW6 Conn_01x02_Male, U1 ATmega8-16PU, U10 74141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

Commit message: Move HV_IN connector to not interfere with NIX1 sub-board.
Parts:
- moved HV_IN1 27.5 mm to (110.5, 189.0), turned to 270 degrees
Routing:
- net Net-(HV_IN1-Pad1): track 156.5 -> 195.0 mm
- net GND: track 464.1 -> 435.1 mm
